Commit message: 1.增加了激光雷达scan的inf数据判定 2.修改OccGridMapBase.h的182来移动地图中心,修改hector_mapping.cc的49、55、57、67、169、175从而修改地图分辨率变化带来的变化。表现：修改分辨率无法显示地图.原因：地图中心偏移，调大分辨率坐标超出量程，从而无法建图

File: urdf/LHD.urdf (robot description, URDF)
Before this commit: robot LHD, 9 links, 8 joints
Links:
- link houcheshen_link: geometry visual mesh filename=package://lesson4/meshes/houcheshen.stl
- link houlun_link: geometry visual mesh filename=package://lesson4/meshes/houlun.stl
- link qiancheshen_link: geometry visual mesh filename=package://lesson4/meshes/qiancheshen.stl
- link qianlun_link: geometry visual mesh filename=package://lesson4/meshes/qianlun.stl

File: urdf/lhd_md1.urdf (robot description, URDF)
Before this commit: robot LHD_md, 10 links, 9 joints
Links:
- link houcheshen_link: geometry visual mesh filename=package://lesson4/meshes/houcheshen.stl
- link houlun_link: geometry visual mesh filename=package://lesson4/meshes/houlun.stl
- link qiancheshen_link: geometry visual mesh filename=package://lesson4/meshes/qiancheshen.stl
- link qianlun_link: geometry visual mesh filename=package://lesson4/meshes/qianlun.stl
